File: Electronique/Carte/carte_1A_cdfr2018.sch (KiCad schematic (older format))
At the start: 25 parts, among them J1 CONN_01X01_GND, J10 Conn_01x02, J11 Conn_01x02, J12 Conn_01x02, J2 CONN_01X01_BATT, J3 CONN_01X01_+7V4, J4 CONN_01X01_+5V, J5 Conn_01x04, J6 Conn_01x04, J7 Conn_01x02, J8 Conn_01x02, J9 Conn_01x02, U1 trou-d3mm, U2 trou-d3mm, U3 trou-d3mm, U4 trou-d3mm, U5 Nucleo-64, U6 Stepstick_gros, U7 Stepstick_gros

Commit message: Electronique
Parts:
- removed J10, J11, J12, J7, J8, J9: Conn_01x02, symbol Conn_01x02
- removed J5, J6: Conn_01x04, symbol Conn_01x04
- removed R4, R5, R6, R7, R8, R9: 10k, symbol R
- removed U6, U7: Stepstick_gros, symbol Stepstick_gros
- added H? (x2): pont_en_H, symbol pont_en_H
- added J5, J6, J?: CONN_01X01_GND, Measurement_Points:Measurement_Point_Round-TH_Big, symbol CONN_01X01
- added N?: SN74HC04N, Housings_DIP:DIP-14_W7.62mm_LongPads, symbol SN74HC04N
- added P1: Encodeur1, Connectors_Molex:Molex_KK-6410-04_04x2.54mm_Straight, symbol CONN_01X04
- added P2: Encodeur2, Connectors_Molex:Molex_KK-6410-04_04x2.54mm_Straight, symbol CONN_01X04
- added P?: ultrason, Connectors_Molex:Molex_KK-6410-04_04x2.54mm_Straight, symbol CONN_01X04
- added P?: servo1, symbol CONN_01X03
- added P?: servo2, symbol CONN_01X03
- added P?: servo3, symbol CONN_01X03
- added R?: R, symbol R
- added T? (x2): SN74LS126AN, Housings_DIP:DIP-14_W7.62mm_LongPads, symbol SN74LS126AN
Connections:
- net labels added: +12V, +12V_P, +20V, +20V_P, +3V3_P, 5V_P, 7V4_P, CH_A1, CH_A2, CH_B1, CH_B2, CodeurEchantillon, Lanceur, RDD, RDG, RGD, RGG, arduinoRX, baliseRX, servo, servoRX, servoTX, ultrason1, ultrason2
- net labels removed: 1A, 2A, BATT_P, C-1, C-2, C-3, dist_1, dist_2, dist_3, dist_4, fc_1, fc_2, fc_3, fc_4, jack, selec, select
- wire segments 135 -> 87
- no-connect marks 50 -> 89

Commit message: kicadFinal
Parts:
- removed H?: pont_en_H, symbol pont_en_H
- H1: renamed from H?; footprint (none) -> robot1A:pont_en_H
- gave numbers to parts that had none: 8
Connections:
- net RDD: now also U5.46 (PB14); no longer U5.6 (PC15)
- net RDG: now also U5.45 (PB13); no longer U5.7 (PC14)
- net RGD: now also U5.54 (PA12); no longer U5.4 (PF1)
- net RGG: now also U5.47 (PB15); no longer U5.5 (PF0)
- net ultrason1: now also U5.78 (PB8); no longer U5.13 (PA13)
- net ultrason2: now also U5.77 (PB9); no longer U5.12 (PA14)
- net +20V renamed +15V
- no-connect marks 89 -> 81

Commit message: rapide corretion des empreintes pour les servos
Parts:
- P4, P5, P6: footprint (none) -> Connectors_Molex:Molex_KK-6410-03_03x2.54mm_Straight
- renumbered R6 to R1, U5 to U1, U1 to U2, U2 to U3, U3 to U4, U4 to U5
Changed lines of the file:
@@
 NoConn ~ 10200 10150
 $Comp
-L PWR_FLAG #FLG01
+L PWR_FLAG #FLG5
 U 1 1 59198CA2
 P 4100 1250
-F 0 "#FLG01" H 4100 1325 50  0001 C CNN
+F 0 "#FLG5" H 4100 1325 50  0001 C CNN
 F 1 "PWR_FLAG" H 4100 1400 50  0000 C CNN
 F 2 "" H 4100 1250 50  0001 C CNN
@@
 NoConn ~ 17300 10350
 $Comp
-L trou-d3mm U1
+L trou-d3mm U2
 U 1 1 591A6CA7
 P 11200 1550
-F 0 "U1" H 11200 1550 60  0000 C CNN
+F 0 "U2" H 11200 1550 60  0000 C CNN
 F 1 "trou-d3mm" H 11250 1650 60  0000 C CNN
 F 2 "robot_1A:trou_d3mm" H 11200 1550 60  0001 C CNN
@@
 $EndComp
 $Comp
-L trou-d3mm U2
+L trou-d3mm U3
 U 1 1 591A6F1E
 P 12150 1550
-F 0 "U2" H 12150 1550 60  0000 C CNN
+F 0 "U3" H 12150 1550 60  0000 C CNN
 F 1 "trou-d3mm" H 12200 1650 60  0000 C CNN
 F 2 "robot_1A:trou_d3mm" H 12150 1550 60  0001 C CNN
@@
 $EndComp
 $Comp
-L trou-d3mm U3
+L trou-d3mm U4
 U 1 1 591A6FB3
 P 13100 1550
-F 0 "U3" H 13100 1550 60  0000 C CNN
+F 0 "U4" H 13100 1550 60  0000 C CNN
 F 1 "trou-d3mm" H 13150 1650 60  0000 C CNN
 F 2 "robot_1A:trou_d3mm" H 13100 1550 60  0001 C CNN
@@
 BATT
 $Comp
-L PWR_FLAG #FLG02
+L PWR_FLAG #FLG6
 U 1 1 5A650CF3
 P 4900 1250
-F 0 "#FLG02" H 4900 1325 50  0001 C CNN
+F 0 "#FLG6" H 4900 1325 50  0001 C CNN
 F 1 "PWR_FLAG" H 4900 1400 50  0000 C CNN
 F 2 "" H 4900 1250 50  0001 C CNN
@@
 +7V4
 $Comp
-L PWR_FLAG #FLG03
+L PWR_FLAG #FLG9
 U 1 1 5A650DA2
 P 5700 1250
-F 0 "#FLG03" H 5700 1325 50  0001 C CNN
+F 0 "#FLG9" H 5700 1325 50  0001 C CNN
 F 1 "PWR_FLAG" H 5700 1400 50  0000 C CNN
 F 2 "" H 5700 1250 50  0001 C CNN
@@
 +5V
 $Comp
-L PWR_FLAG #FLG04
+L PWR_FLAG #FLG10
 U 1 1 5A650E4F
 P 6500 1250
-F 0 "#FLG04" H 6500 1325 50  0001 C CNN
+F 0 "#FLG10" H 6500 1325 50  0001 C CNN
 F 1 "PWR_FLAG" H 6500 1400 50  0000 C CNN
 F 2 "" H 6500 1250 50  0001 C CNN
@@
 +3V3
 $Comp
-L trou-d3mm U4
+L trou-d3mm U5
 U 1 1 5A65AF33
 P 14050 1550
-F 0 "U4" H 14050 1550 60  0000 C CNN
+F 0 "U5" H 14050 1550 60  0000 C CNN
 F 1 "trou-d3mm" H 14100 1650 60  0000 C CNN
 F 2 "robot_1A:trou_d3mm" H 14050 1550 60  0001 C CNN
@@
 NoConn ~ 10200 10350
 $Comp
-L Nucleo-64 U5
+L Nucleo-64 U1
 U 1 1 591611DF
 P 9150 14150
-F 0 "U5" H 9200 14200 60  0000 C CNN
+F 0 "U1" H 9200 14200 60  0000 C CNN
 F 1 "Nucleo-64" H 13500 23150 100 0000 C CNN
 F 2 "robot_1A:Nucleo-64" H 13400 25600 60  0001 C CNN
@@
 Lanceur
 $Comp
-L PWR_FLAG #FLG05
+L PWR_FLAG #FLG20
 U 1 1 5ABE4366
 P 17450 6350
-F 0 "#FLG05" H 17450 6425 50  0001 C CNN
+F 0 "#FLG20" H 17450 6425 50  0001 C CNN
 F 1 "PWR_FLAG" H 17450 6500 50  0000 C CNN
 F 2 "" H 17450 6350 50  0001 C CNN
@@
 $EndComp
 $Comp
-L PWR_FLAG #FLG06
+L PWR_FLAG #FLG19
 U 1 1 5ABE4399
 P 17450 6150
-F 0 "#FLG06" H 17450 6225 50  0001 C CNN
+F 0 "#FLG19" H 17450 6225 50  0001 C CNN
 F 1 "PWR_FLAG" H 17450 6300 50  0000 C CNN
 F 2 "" H 17450 6150 50  0001 C CNN
@@
 $EndComp
 $Comp
-L PWR_FLAG #FLG07
+L PWR_FLAG #FLG18
 U 1 1 5ABE43C5
 P 17450 5950
-F 0 "#FLG07" H 17450 6025 50  0001 C CNN
+F 0 "#FLG18" H 17450 6025 50  0001 C CNN
 F 1 "PWR_FLAG" H 17450 6100 50  0000 C CNN
 F 2 "" H 17450 5950 50  0001 C CNN
@@
 $EndComp
 $Comp
-L PWR_FLAG #FLG08
+L PWR_FLAG #FLG17
 U 1 1 5ABE43F1
 P 17450 4550
-F 0 "#FLG08" H 17450 4625 50  0001 C CNN
+F 0 "#FLG17" H 17450 4625 50  0001 C CNN
 F 1 "PWR_FLAG" H 17450 4700 50  0000 C CNN
 F 2 "" H 17450 4550 50  0001 C CNN
@@
 $EndComp
 $Comp
-L PWR_FLAG #FLG09
+L PWR_FLAG #FLG14
 U 1 1 5ABE441D
 P 10050 6950
-F 0 "#FLG09" H 10050 7025 50  0001 C CNN
+F 0 "#FLG14" H 10050 7025 50  0001 C CNN
 F 1 "PWR_FLAG" H 10050 7100 50  0000 C CNN
 F 2 "" H 10050 6950 50  0001 C CNN
@@
 servo
 $Comp
-L PWR_FLAG #FLG010
+L PWR_FLAG #FLG15
 U 1 1 5ABFC66C
 P 10050 7150
-F 0 "#FLG010" H 10050 7225 50  0001 C CNN
+F 0 "#FLG15" H 10050 7225 50  0001 C CNN
 F 1 "PWR_FLAG" H 10050 7300 50  0000 C CNN
 F 2 "" H 10050 7150 50  0001 C CNN
@@
 +12V
 $Comp
-L PWR_FLAG #FLG011
+L PWR_FLAG #FLG11
 U 1 1 5AC0B6C0
 P 7300 1250
-F 0 "#FLG011" H 7300 1325 50  0001 C CNN
+F 0 "#FLG11" H 7300 1325 50  0001 C CNN
 F 1 "PWR_FLAG" H 7300 1400 50  0000 C CNN
 F 2 "" H 7300 1250 50  0001 C CNN
@@
 +15V
 $Comp
-L PWR_FLAG #FLG012
+L PWR_FLAG #FLG12
 U 1 1 5AC0B7B7
 P 8100 1250
-F 0 "#FLG012" H 8100 1325 50  0001 C CNN
+F 0 "#FLG12" H 8100 1325 50  0001 C CNN
 F 1 "PWR_FLAG" H 8100 1400 50  0000 C CNN
 F 2 "" H 8100 1250 50  0001 C CNN
@@
 	3050 8550 3050 8700
 $Comp
-L PWR_FLAG #FLG013
+L PWR_FLAG #FLG3
 U 1 1 5AC151C9
 P 3550 9700
-F 0 "#FLG013" H 3550 9775 50  0001 C CNN
+F 0 "#FLG3" H 3550 9775 50  0001 C CNN
 F 1 "PWR_FLAG" H 3550 9850 50  0000 C CNN
 F 2 "" H 3550 9700 50  0001 C CNN
@@
 $EndComp
 $Comp
-L PWR_FLAG #FLG014
+L PWR_FLAG #FLG4
 U 1 1 5AC15208
 P 3550 9900
-F 0 "#FLG014" H 3550 9975 50  0001 C CNN
+F 0 "#FLG4" H 3550 9975 50  0001 C CNN
 F 1 "PWR_FLAG" H 3550 10050 50  0000 C CNN
 F 2 "" H 3550 9900 50  0001 C CNN
@@
 $EndComp
 $Comp
-L PWR_FLAG #FLG015
+L PWR_FLAG #FLG1
 U 1 1 5AC1524F
 P 3550 8800
-F 0 "#FLG015" H 3550 8875 50  0001 C CNN
+F 0 "#FLG1" H 3550 8875 50  0001 C CNN
 F 1 "PWR_FLAG" H 3550 8950 50  0000 C CNN
 F 2 "" H 3550 8800 50  0001 C CNN
@@
 $EndComp
 $Comp
-L PWR_FLAG #FLG016
+L PWR_FLAG #FLG2
 U 1 1 5AC15287
 P 3550 9000
-F 0 "#FLG016" H 3550 9075 50  0001 C CNN
+F 0 "#FLG2" H 3550 9075 50  0001 C CNN
 F 1 "PWR_FLAG" H 3550 9150 50  0000 C CNN
 F 2 "" H 3550 9000 50  0001 C CNN
@@
 	17600 9350 17300 9350
 $Comp
-L PWR_FLAG #FLG017
+L PWR_FLAG #FLG16
 U 1 1 5AC16DBB
 P 10100 10750
-F 0 "#FLG017" H 10100 10825 50  0001 C CNN
+F 0 "#FLG16" H 10100 10825 50  0001 C CNN
 F 1 "PWR_FLAG" H 10100 10900 50  0000 C CNN
 F 2 "" H 10100 10750 50  0001 C CNN
@@
 $EndComp
 $Comp
-L PWR_FLAG #FLG018
+L PWR_FLAG #FLG13
 U 1 1 5AC64DBF
 P 8900 1250
-F 0 "#FLG018" H 8900 1325 50  0001 C CNN
+F 0 "#FLG13" H 8900 1325 50  0001 C CNN
 F 1 "PWR_FLAG" H 8900 1400 50  0000 C CNN
 F 2 "" H 8900 1250 50  0001 C CNN
@@
 5V_P
 $Comp
-L GND #PWR019
+L GND #PWR1
 U 1 1 5AC669B4
 P 5050 9200
-F 0 "#PWR019" H 5050 8950 50  0001 C CNN
+F 0 "#PWR1" H 5050 8950 50  0001 C CNN
 F 1 "GND" H 5050 9050 50  0000 C CNN
 F 2 "" H 5050 9200 50  0001 C CNN
@@
 ultrason2
 $Comp
-L PWR_FLAG #FLG020
+L PWR_FLAG #FLG7
 U 1 1 5AC66D24
 P 5350 8850
-F 0 "#FLG020" H 5350 8925 50  0001 C CNN
+F 0 "#FLG7" H 5350 8925 50  0001 C CNN
 F 1 "PWR_FLAG" H 5350 9000 50  0000 C CNN
 F 2 "" H 5350 8850 50  0001 C CNN
@@
 $EndComp
 $Comp
-L PWR_FLAG #FLG021
+L PWR_FLAG #FLG8
 U 1 1 5AC66DB1
 P 5350 8950
-F 0 "#FLG021" H 5350 9025 50  0001 C CNN
+F 0 "#FLG8" H 5350 9025 50  0001 C CNN
 F 1 "PWR_FLAG" H 5350 9100 50  0000 C CNN
 F 2 "" H 5350 8950 50  0001 C CNN
@@
 F 0 "P4" H 23100 8900 50  0000 C CNN
 F 1 "servo1" V 23200 8700 50  0000 C CNN
-F 2 "" H 23100 8700 50  0000 C CNN
+F 2 "Connectors_Molex:Molex_KK-6410-03_03x2.54mm_Straight" H 23100 8700 50  0000 C CNN
 F 3 "" H 23100 8700 50  0000 C CNN
 	1    23100 8700
@@
 F 0 "P5" H 23100 9450 50  0000 C CNN
 F 1 "servo2" V 23200 9250 50  0000 C CNN
-F 2 "" H 23100 9250 50  0000 C CNN
+F 2 "Connectors_Molex:Molex_KK-6410-03_03x2.54mm_Straight" H 23100 9250 50  0000 C CNN
 F 3 "" H 23100 9250 50  0000 C CNN
 	1    23100 9250
@@
 F 0 "P6" H 23100 9950 50  0000 C CNN
 F 1 "servo3" V 23200 9750 50  0000 C CNN
-F 2 "" H 23100 9750 50  0000 C CNN
+F 2 "Connectors_Molex:Molex_KK-6410-03_03x2.54mm_Straight" H 23100 9750 50  0000 C CNN
 F 3 "" H 23100 9750 50  0000 C CNN
 	1    23100 9750
@@
 7V4_P
 $Comp
-L GND #PWR022
+L GND #PWR5
 U 1 1 5AC690E5
 P 22900 8600
-F 0 "#PWR022" H 22900 8350 50  0001 C CNN
+F 0 "#PWR5" H 22900 8350 50  0001 C CNN
 F 1 "GND" H 22900 8450 50  0000 C CNN
 F 2 "" H 22900 8600 50  0001 C CNN
@@
 7V4_P
 $Comp
-L GND #PWR023
+L GND #PWR6
 U 1 1 5AC6915C
 P 22900 9150
-F 0 "#PWR023" H 22900 8900 50  0001 C CNN
+F 0 "#PWR6" H 22900 8900 50  0001 C CNN
 F 1 "GND" H 22900 9000 50  0000 C CNN
 F 2 "" H 22900 9150 50  0001 C CNN
@@
 7V4_P
 $Comp
-L GND #PWR024
+L GND #PWR7
 U 1 1 5AC691B5
 P 22900 9650
-F 0 "#PWR024" H 22900 9400 50  0001 C CNN
+F 0 "#PWR7" H 22900 9400 50  0001 C CNN
 F 1 "GND" H 22900 9500 50  0000 C CNN
 F 2 "" H 22900 9650 50  0001 C CNN
@@
 	19750 11200 20250 11200
 $Comp
-L GND #PWR025
+L GND #PWR4
 U 1 1 5AC721A8
 P 20250 12000
-F 0 "#PWR025" H 20250 11750 50  0001 C CNN
+F 0 "#PWR4" H 20250 11750 50  0001 C CNN
 F 1 "GND" H 20250 11850 50  0000 C CNN
 F 2 "" H 20250 12000 50  0001 C CNN
@@
 $EndComp
 $Comp
-L GND #PWR026
+L GND #PWR3
 U 1 1 5AC72214
 P 20150 9450
-F 0 "#PWR026" H 20150 9200 50  0001 C CNN
+F 0 "#PWR3" H 20150 9200 50  0001 C CNN
 F 1 "GND" H 20150 9300 50  0000 C CNN
 F 2 "" H 20150 9450 50  0001 C CNN
@@
 +5V_P
 $Comp
-L R R6
+L R R1
 U 1 1 5AC74808
 P 21850 8600
-F 0 "R6" V 21930 8600 50  0000 C CNN
+F 0 "R1" V 21930 8600 50  0000 C CNN
 F 1 "R" V 21850 8600 50  0000 C CNN
 F 2 "" V 21780 8600 50  0001 C CNN
@@
 	20800 10550 20700 10550
 $Comp
-L GND #PWR027
+L GND #PWR2
 U 1 1 5AC75453
 P 20000 10500
-F 0 "#PWR027" H 20000 10250 50  0001 C CNN
+F 0 "#PWR2" H 20000 10250 50  0001 C CNN
 F 1 "GND" H 20000 10350 50  0000 C CNN
 F 2 "" H 20000 10500 50  0001 C CNN

Commit message: Kicad Final enfin !!
Parts:
- removed J7: CONN_01X01_GND, Measurement_Points:Measurement_Point_Round-TH_Big, symbol CONN_01X01
- added P3, P5, P6: ultrason, Connectors_Molex:Molex_KK-6410-04_04x2.54mm_Straight, symbol CONN_01X04
- R1: footprint (none) -> Resistors_SMD:R_1206_HandSoldering
- renumbered P3 to P4, P4 to P7, P5 to P8, P6 to P9
Connections:
- net +12V is gone; now on net +12V_P: J5.1 (P1)
- net +5V is gone; now on net +5V_P: J4.1 (P1)
- net 5V_P: now also P3.4 (P4), P5.4 (P4), P6.4 (P4)
- net GND: now also P3.1 (P1), P5.1 (P1), P6.1 (P1)
- net ultrason4: now reaches U1.21 (PC0)
- net ultrason4: now also P5.2 (P2)
- net ultrason3: now reaches U1.22 (PC1)
- net ultrason3: now also P5.3 (P3)
- net ultrason8: now reaches U1.23 (PB0)
- net ultrason8: now also P6.2 (P2)
- net ultrason5: now reaches U1.43 (PC4)
- net ultrason5: now also P3.3 (P3)
- net ultrason7: now reaches U1.57 (PC5)
- net ultrason7: now also P6.3 (P3)
- net ultrason6: now reaches U1.72 (PA7)
- net ultrason6: now also P3.2 (P2)
- net +15V renamed +15V_P
- net +7V4 renamed +7V4_P
- net BATT renamed BATT_P
- no-connect marks 81 -> 76
