File: Electronique/Carte/file5AC61AC3.sch (KiCad schematic (older format))
At the start: 21 parts

Commit message: kicadFinal
Parts:
- removed C? (x2): C, symbol C
- removed R?: 560R, symbol R
- removed R?: 330R, symbol R
- removed U?: LM317_SOT223, symbol LM317_SOT223
- U10, U11, U12, U13: renamed from U?; footprint (none) -> DSN:DSN2596
- U6, U7, U8, U9: renamed from U?; footprint (none) -> DSN:B plug 5mm
- gave numbers to parts that had none: 7
- renumbered F to F6
Connections:
- net +20V renamed +15V

Commit message: rapide corretion des empreintes pour les servos
Changed lines of the file:
@@
 $EndComp
 $Comp
-L GND #PWR033
+L GND #PWR8
 U 1 1 5AC620F3
 P 1600 2050
-F 0 "#PWR033" H 1600 1800 50  0001 C CNN
+F 0 "#PWR8" H 1600 1800 50  0001 C CNN
 F 1 "GND" H 1600 1900 50  0000 C CNN
 F 2 "" H 1600 2050 50  0001 C CNN
@@
 	1450 1850 1800 1850
 $Comp
-L PWR_FLAG #FLG034
+L PWR_FLAG #FLG26
 U 1 1 5AC62146
 P 2300 1850
-F 0 "#FLG034" H 2300 1925 50  0001 C CNN
+F 0 "#FLG26" H 2300 1925 50  0001 C CNN
 F 1 "PWR_FLAG" H 2300 2000 50  0000 C CNN
 F 2 "" H 2300 1850 50  0001 C CNN
@@
 BATT
 Wire Wire Line
-	2100 1850 2300 1850
-Wire Wire Line
-	2300 1850 2500 1850
-Wire Wire Line
-	2500 1850 3450 1850
+	2100 1850 3450 1850
 Connection ~ 2300 1850
 Wire Wire Line
@@
 Connection ~ 2500 1850
 $Comp
-L GND #PWR035
+L GND #PWR12
 U 1 1 5AC621C7
 P 3250 2150
-F 0 "#PWR035" H 3250 1900 50  0001 C CNN
+F 0 "#PWR12" H 3250 1900 50  0001 C CNN
 F 1 "GND" H 3250 2000 50  0000 C CNN
 F 2 "" H 3250 2150 50  0001 C CNN
@@
 	3250 2050 3450 2050
 $Comp
-L GND #PWR036
+L GND #PWR16
 U 1 1 5AC6235A
 P 4800 2200
-F 0 "#PWR036" H 4800 1950 50  0001 C CNN
+F 0 "#PWR16" H 4800 1950 50  0001 C CNN
 F 1 "GND" H 4800 2050 50  0000 C CNN
 F 2 "" H 4800 2200 50  0001 C CNN
@@
 	4550 1850 5250 1850
 Wire Wire Line
-	5250 1600 5250 1850
-Wire Wire Line
-	5250 1850 5250 1900
-$Comp
-L GND #PWR037
+	5250 1600 5250 1900
+$Comp
+L GND #PWR20
 U 1 1 5AC62460
 P 5250 2350
-F 0 "#PWR037" H 5250 2100 50  0001 C CNN
+F 0 "#PWR20" H 5250 2100 50  0001 C CNN
 F 1 "GND" H 5250 2200 50  0000 C CNN
 F 2 "" H 5250 2350 50  0001 C CNN
@@
 $EndComp
 $Comp
-L GND #PWR038
+L GND #PWR9
 U 1 1 5AC63DE3
 P 1600 3950
-F 0 "#PWR038" H 1600 3700 50  0001 C CNN
+F 0 "#PWR9" H 1600 3700 50  0001 C CNN
 F 1 "GND" H 1600 3800 50  0000 C CNN
 F 2 "" H 1600 3950 50  0001 C CNN
@@
 	1450 3750 1800 3750
 $Comp
-L PWR_FLAG #FLG039
+L PWR_FLAG #FLG27
 U 1 1 5AC63DEC
 P 2300 3750
-F 0 "#FLG039" H 2300 3825 50  0001 C CNN
+F 0 "#FLG27" H 2300 3825 50  0001 C CNN
 F 1 "PWR_FLAG" H 2300 3900 50  0000 C CNN
 F 2 "" H 2300 3750 50  0001 C CNN
@@
 BATT
 Wire Wire Line
-	2100 3750 2300 3750
-Wire Wire Line
-	2300 3750 2500 3750
-Wire Wire Line
-	2500 3750 3450 3750
+	2100 3750 3450 3750
 Connection ~ 2300 3750
 Wire Wire Line
@@
 Connection ~ 2500 3750
 $Comp
-L GND #PWR040
+L GND #PWR13
 U 1 1 5AC63DF7
 P 3250 4050
-F 0 "#PWR040" H 3250 3800 50  0001 C CNN
+F 0 "#PWR13" H 3250 3800 50  0001 C CNN
 F 1 "GND" H 3250 3900 50  0000 C CNN
 F 2 "" H 3250 4050 50  0001 C CNN
@@
 	3250 3950 3450 3950
 $Comp
-L GND #PWR041
+L GND #PWR17
 U 1 1 5AC63DFF
 P 4800 4100
-F 0 "#PWR041" H 4800 3850 50  0001 C CNN
+F 0 "#PWR17" H 4800 3850 50  0001 C CNN
 F 1 "GND" H 4800 3950 50  0000 C CNN
 F 2 "" H 4800 4100 50  0001 C CNN
@@
 	4550 3750 5250 3750
 Wire Wire Line
-	5250 3550 5250 3750
-Wire Wire Line
-	5250 3750 5250 3800
-$Comp
-L GND #PWR042
+	5250 3550 5250 3800
+$Comp
+L GND #PWR21
 U 1 1 5AC63E0F
 P 5250 4250
-F 0 "#PWR042" H 5250 4000 50  0001 C CNN
+F 0 "#PWR21" H 5250 4000 50  0001 C CNN
 F 1 "GND" H 5250 4100 50  0000 C CNN
 F 2 "" H 5250 4250 50  0001 C CNN
@@
 $EndComp
 $Comp
-L GND #PWR043
+L GND #PWR10
 U 1 1 5AC658A5
 P 1600 5350
-F 0 "#PWR043" H 1600 5100 50  0001 C CNN
+F 0 "#PWR10" H 1600 5100 50  0001 C CNN
 F 1 "GND" H 1600 5200 50  0000 C CNN
 F 2 "" H 1600 5350 50  0001 C CNN
@@
 	1450 5150 1800 5150
 $Comp
-L PWR_FLAG #FLG044
+L PWR_FLAG #FLG28
 U 1 1 5AC658AE
 P 2300 5150
-F 0 "#FLG044" H 2300 5225 50  0001 C CNN
+F 0 "#FLG28" H 2300 5225 50  0001 C CNN
 F 1 "PWR_FLAG" H 2300 5300 50  0000 C CNN
 F 2 "" H 2300 5150 50  0001 C CNN
@@
 BATT
 Wire Wire Line
-	2100 5150 2300 5150
-Wire Wire Line
-	2300 5150 2500 5150
-Wire Wire Line
-	2500 5150 3450 5150
+	2100 5150 3450 5150
 Connection ~ 2300 5150
 Wire Wire Line
@@
 Connection ~ 2500 5150
 $Comp
-L GND #PWR045
+L GND #PWR14
 U 1 1 5AC658B9
 P 3250 5450
-F 0 "#PWR045" H 3250 5200 50  0001 C CNN
+F 0 "#PWR14" H 3250 5200 50  0001 C CNN
 F 1 "GND" H 3250 5300 50  0000 C CNN
 F 2 "" H 3250 5450 50  0001 C CNN
@@
 	3250 5350 3450 5350
 $Comp
-L GND #PWR046
+L GND #PWR18
 U 1 1 5AC658C1
 P 4800 5500
-F 0 "#PWR046" H 4800 5250 50  0001 C CNN
+F 0 "#PWR18" H 4800 5250 50  0001 C CNN
 F 1 "GND" H 4800 5350 50  0000 C CNN
 F 2 "" H 4800 5500 50  0001 C CNN
@@
 	4550 5150 5250 5150
 Wire Wire Line
-	5250 4950 5250 5150
-Wire Wire Line
-	5250 5150 5250 5200
-$Comp
-L GND #PWR047
+	5250 4950 5250 5200
+$Comp
+L GND #PWR22
 U 1 1 5AC658D1
 P 5250 5650
-F 0 "#PWR047" H 5250 5400 50  0001 C CNN
+F 0 "#PWR22" H 5250 5400 50  0001 C CNN
 F 1 "GND" H 5250 5500 50  0000 C CNN
 F 2 "" H 5250 5650 50  0001 C CNN
@@
 $EndComp
 $Comp
-L GND #PWR048
+L GND #PWR11
 U 1 1 5AC65C25
 P 1600 6800
-F 0 "#PWR048" H 1600 6550 50  0001 C CNN
+F 0 "#PWR11" H 1600 6550 50  0001 C CNN
 F 1 "GND" H 1600 6650 50  0000 C CNN
 F 2 "" H 1600 6800 50  0001 C CNN
@@
 	1450 6600 1800 6600
 $Comp
-L PWR_FLAG #FLG049
+L PWR_FLAG #FLG29
 U 1 1 5AC65C2E
 P 2300 6600
-F 0 "#FLG049" H 2300 6675 50  0001 C CNN
+F 0 "#FLG29" H 2300 6675 50  0001 C CNN
 F 1 "PWR_FLAG" H 2300 6750 50  0000 C CNN
 F 2 "" H 2300 6600 50  0001 C CNN
@@
 BATT
 Wire Wire Line
-	2100 6600 2300 6600
-Wire Wire Line
-	2300 6600 2500 6600
-Wire Wire Line
-	2500 6600 3450 6600
+	2100 6600 3450 6600
 Connection ~ 2300 6600
 Wire Wire Line
@@
 Connection ~ 2500 6600
 $Comp
-L GND #PWR050
+L GND #PWR15
 U 1 1 5AC65C39
 P 3250 6900
-F 0 "#PWR050" H 3250 6650 50  0001 C CNN
+F 0 "#PWR15" H 3250 6650 50  0001 C CNN
 F 1 "GND" H 3250 6750 50  0000 C CNN
 F 2 "" H 3250 6900 50  0001 C CNN
@@
 	3250 6800 3450 6800
 $Comp
-L GND #PWR051
+L GND #PWR19
 U 1 1 5AC65C41
 P 4800 6950
-F 0 "#PWR051" H 4800 6700 50  0001 C CNN
+F 0 "#PWR19" H 4800 6700 50  0001 C CNN
 F 1 "GND" H 4800 6800 50  0000 C CNN
 F 2 "" H 4800 6950 50  0001 C CNN
@@
 	4550 6600 5250 6600
 Wire Wire Line
-	5250 6400 5250 6600
-Wire Wire Line
-	5250 6600 5250 6650
-$Comp
-L GND #PWR052
+	5250 6400 5250 6650
+$Comp
+L GND #PWR23
 U 1 1 5AC65C51
 P 5250 7100
-F 0 "#PWR052" H 5250 6850 50  0001 C CNN
+F 0 "#PWR23" H 5250 6850 50  0001 C CNN
 F 1 "GND" H 5250 6950 50  0000 C CNN
 F 2 "" H 5250 7100 50  0001 C CNN

Commit message: correction
Parts:
- removed U13: DSN2596, DSN:DSN2596, symbol DSN2596
- added U10, U14: B_Plug_5mm, dsn2596:B plug 5mm, symbol B_Plug_5mm
- C1, C2, C3, C4: footprint (none) -> Capacitors_THT:CP_Radial_D8.0mm_P3.50mm
- renumbered U10 to U11, U11 to U12, U12 to U13
Connections:
- net +15V: now also U14.1
- net BATT: now also U10.2
- net GND: now also U10.1, U14.2
Changed lines of the file:
@@
 $EndDescr
 $Comp
-L DSN2596 U10
+L DSN2596 U11
 U 1 1 5AC61E96
 P 4000 1950
-F 0 "U10" H 3700 2200 60  0000 C CNN
+F 0 "U11" H 3700 2200 60  0000 C CNN
 F 1 "DSN2596" H 3850 2300 60  0000 C CNN
 F 2 "DSN:DSN2596" H 4000 1950 60  0000 C CNN
@@
 F 0 "C1" H 5275 2150 50  0000 L CNN
 F 1 "CP" H 5275 1950 50  0000 L CNN
-F 2 "" H 5288 1900 50  0001 C CNN
+F 2 "Capacitors_THT:CP_Radial_D8.0mm_P3.50mm" H 5288 1900 50  0001 C CNN
 F 3 "" H 5250 2050 50  0001 C CNN
 	1    5250 2050
@@
 	5250 2200 5250 2350
 $Comp
-L DSN2596 U11
+L DSN2596 U12
 U 1 1 5AC63DD1
 P 4000 3850
-F 0 "U11" H 3700 4100 60  0000 C CNN
+F 0 "U12" H 3700 4100 60  0000 C CNN
 F 1 "DSN2596" H 3850 4200 60  0000 C CNN
 F 2 "DSN:DSN2596" H 4000 3850 60  0000 C CNN
@@
 F 0 "C2" H 5275 4050 50  0000 L CNN
 F 1 "CP" H 5275 3850 50  0000 L CNN
-F 2 "" H 5288 3800 50  0001 C CNN
+F 2 "Capacitors_THT:CP_Radial_D8.0mm_P3.50mm" H 5288 3800 50  0001 C CNN
 F 3 "" H 5250 3950 50  0001 C CNN
 	1    5250 3950
@@
 Connection ~ 5250 1850
 $Comp
-L DSN2596 U12
+L DSN2596 U13
 U 1 1 5AC65893
 P 4000 5250
-F 0 "U12" H 3700 5500 60  0000 C CNN
+F 0 "U13" H 3700 5500 60  0000 C CNN
 F 1 "DSN2596" H 3850 5600 60  0000 C CNN
 F 2 "DSN:DSN2596" H 4000 5250 60  0000 C CNN
@@
 F 0 "C3" H 5275 5450 50  0000 L CNN
 F 1 "CP" H 5275 5250 50  0000 L CNN
-F 2 "" H 5288 5200 50  0001 C CNN
+F 2 "Capacitors_THT:CP_Radial_D8.0mm_P3.50mm" H 5288 5200 50  0001 C CNN
 F 3 "" H 5250 5350 50  0001 C CNN
 	1    5250 5350
@@
 +12V
 Connection ~ 5250 5150
-$Comp
-L DSN2596 U13
-U 1 1 5AC65C13
-P 4000 6700
-F 0 "U13" H 3700 6950 60  0000 C CNN
-F 1 "DSN2596" H 3850 7050 60  0000 C CNN
-F 2 "DSN:DSN2596" H 4000 6700 60  0000 C CNN
-F 3 "" H 4000 6700 60  0000 C CNN
-	1    4000 6700
-	1    0    0    -1
-$EndComp
 $Comp
 L B_Plug_5mm U9
@@
 F 0 "C4" H 5275 6900 50  0000 L CNN
 F 1 "CP" H 5275 6700 50  0000 L CNN
-F 2 "" H 5288 6650 50  0001 C CNN
+F 2 "Capacitors_THT:CP_Radial_D8.0mm_P3.50mm" H 5288 6650 50  0001 C CNN
 F 3 "" H 5250 6800 50  0001 C CNN
 	1    5250 6800
@@
 +15V
 Connection ~ 5250 6600
+$Comp
+L B_Plug_5mm U10
+U 1 1 5ACA92D8
+P 3650 6700
+F 0 "U10" H 3650 7100 60  0000 C CNN
+F 1 "B_Plug_5mm" H 3650 7200 60  0000 C CNN
+F 2 "dsn2596:B plug 5mm" H 3650 6700 60  0000 C CNN
+F 3 "" H 3650 6700 60  0000 C CNN
+	1    3650 6700
+	-1   0    0    1
+$EndComp
+$Comp
+L B_Plug_5mm U14
+U 1 1 5ACA93FA
+P 4350 6700
+F 0 "U14" H 4350 7100 60  0000 C CNN
+F 1 "B_Plug_5mm" H 4350 7200 60  0000 C CNN
+F 2 "dsn2596:B plug 5mm" H 4350 6700 60  0000 C CNN
+F 3 "" H 4350 6700 60  0000 C CNN
+	1    4350 6700
+	1    0    0    -1
+$EndComp
+Wire Wire Line
+	3450 6600 3450 6650
+Wire Wire Line
+	3450 6650 3550 6650
+Wire Wire Line
+	3550 6750 3450 6750
+Wire Wire Line
+	3450 6750 3450 6800
+Wire Wire Line
+	4550 6600 4550 6650
+Wire Wire Line
+	4550 6650 4450 6650
+Wire Wire Line
+	4450 6750 4550 6750
+Wire Wire Line
+	4550 6750 4550 6800
 $EndSCHEMATC

Commit message: Kicad Final enfin !!
Parts:
- removed F7, F8, F9: Fuse, Fuse_Holders_and_Fuses:Fuseholder5x20_horiz_SemiClosed_Casing10x25mm, symbol Fuse
- removed U7, U8, U9: B_Plug_5mm, DSN:B plug 5mm, symbol B_Plug_5mm
- renumbered U13 to U10, U14 to U11, U10 to U7, U11 to U8, U12 to U9
